Commit message: Added meshes

File: vention_rail_description/urdf/vention_macro.urdf.xacro (robot description, xacro)
@@ -9,25 +9,30 @@
     position_limit:=2.0
     velocity_limit:=0.5">
-    <link name="${tf_prefix}base_link">
+    <link name="${tf_prefix}vention_rail_base_link">
       <visual>
         <origin xyz="-1.18125 0 0" rpy="0 0 0"/>
         <geometry>
-          <box size="2.3625 0.153 0.09"/>
+          <!-- <box size="2.3625 0.153 0.09"/> -->
+          <mesh filename="file://$(find vention_rail_description)/meshes/base.dae"/>
         </geometry>
       </visual>
     </link>
-    <link name="${tf_prefix}carriage">
+    <link name="${tf_prefix}vention_rail_carriage">
       <visual>
-        <origin xyz="-0.1115 0 0.0565" rpy="0 0 0"/>
+        <origin xyz="-0.1115 0 0.39115" rpy="0 0 0"/>
         <geometry>
           <box size="0.223 0.223 0.023"/>
+          <!-- <mesh filename="file://$(find vention_rail_description)/meshes/carriage.dae"/> -->
         </geometry>
+        <material name="grey">
+          <color rgba="0.7 0.7 0.7 1"/>
+        </material>
       </visual>
     </link>
-    <joint name="${tf_prefix}base_to_carriage" type="prismatic">
+    <joint name="${tf_prefix}vention_rail_base_to_carriage" type="prismatic">
       <origin xyz="-0.223 0 0" rpy="0 0 3.14159"/>
-      <parent link="${tf_prefix}base_link"/>
-      <child link="${tf_prefix}carriage"/>
-      <limit effort="1000" velocity="0.197" lower="0" upper="2.1395"/>
+      <parent link="${tf_prefix}vention_rail_base_link"/>
+      <child link="${tf_prefix}vention_rail_carriage"/>
+      <limit effort="1000" velocity="${velocity_limit}" lower="0" upper="${position_limit}"/>
     </joint>
     <xacro:include filename="$(find vention_rail_description)/urdf/vention_rail.ros2_control.xacro" />

File: vention_rail_description/urdf/vention_rail.ros2_control.xacro (robot description, xacro)
@@ -19,5 +19,5 @@
                     <param name="velocity_limit">${velocity_limit}</param>
                 </hardware>
-                <joint name="${tf_prefix}base_to_carriage">
+                <joint name="${tf_prefix}vention_rail_base_to_carriage">
                     <command_interface name="position"/>
                     <state_interface name="position"/>
@@ -32,5 +32,5 @@
                     <plugin>mock_components/GenericSystem</plugin>
                 </hardware>
-                <joint name="${tf_prefix}base_to_carriage">
+                <joint name="${tf_prefix}vention_rail_base_to_carriage">
                 <command_interface name="position">
                     <param name="min">0</param>

Commit message: meshes with fixed links added, need to unfix links and add inertial data

File: vention_rail_description/urdf/vention_macro.urdf.xacro (robot description, xacro)
@@ -11,28 +11,68 @@
     <link name="${tf_prefix}vention_rail_base_link">
       <visual>
-        <origin xyz="-1.18125 0 0" rpy="0 0 0"/>
+        <origin xyz="0 0 0.045" rpy="0 0 0"/>
         <geometry>
-          <!-- <box size="2.3625 0.153 0.09"/> -->
-          <mesh filename="file://$(find vention_rail_description)/meshes/base.dae"/>
+          <mesh filename="file://$(find vention_rail_description)/meshes/rail_des_live_body.dae"/>
         </geometry>
       </visual>
+      <collision>
+        <origin xyz="-0.0375 0 0.045" rpy="0 0 0"/>
+        <geometry>
+          <box size="2.4375 0.1350 0.0900"/>
+        </geometry>
+      </collision>
     </link>
     <link name="${tf_prefix}vention_rail_carriage">
       <visual>
-        <origin xyz="-0.1115 0 0.39115" rpy="0 0 0"/>
         <geometry>
-          <box size="0.223 0.223 0.023"/>
-          <!-- <mesh filename="file://$(find vention_rail_description)/meshes/carriage.dae"/> -->
+          <mesh filename="file://$(find vention_rail_description)/meshes/rail_des_live_carriage.dae"/>
         </geometry>
-        <material name="grey">
-          <color rgba="0.7 0.7 0.7 1"/>
-        </material>
       </visual>
+      <collision>
+        <origin xyz="0 0 0.00825" rpy="0 0 0"/>
+        <geometry>
+          <box size="0.223 0.223 0.0205000"/>
+        </geometry>
+      </collision>
     </link>
-    <joint name="${tf_prefix}vention_rail_base_to_carriage" type="prismatic">
-      <origin xyz="-0.223 0 0" rpy="0 0 3.14159"/>
+    <joint name="vention_rail_base_to_carriage" type="fixed">
+      <origin xyz="-0.96975 0 0.09600" rpy="0 0 0"/>
       <parent link="${tf_prefix}vention_rail_base_link"/>
       <child link="${tf_prefix}vention_rail_carriage"/>
-      <limit effort="1000" velocity="${velocity_limit}" lower="0" upper="${position_limit}"/>
+    </joint>
+    <link name="${tf_prefix}vention_rail_gearbox">
+      <visual>
+        <geometry>
+          <mesh filename="file://$(find vention_rail_description)/meshes/rail_des_gearbox.dae"/>
+        </geometry>
+      </visual>
+      <collision>
+        <origin xyz="0.013 0 0.017875" rpy="0 0 0"/>
+        <geometry>
+          <box size="0.12310 0.08600 0.13735"/>
+        </geometry>
+      </collision>
+    </link>
+    <joint name="vention_rail_base_to_gearbox" type="fixed">
+      <origin xyz="-1.3308 0 0.05455" rpy="0 0 0"/>
+      <parent link="${tf_prefix}vention_rail_base_link"/>
+      <child link="${tf_prefix}vention_rail_gearbox"/>
+    </joint>
+    <link name="vention_rail_motor">
+      <visual>
+        <geometry>
+          <box size="0.086 0.086 0.226"/>
+        </geometry>
+      </visual>
+      <collision>
+        <geometry>
+          <box size="0.086 0.086 0.226"/>
+        </geometry>
+      </collision>
+    </link>
+    <joint name="vention_rail_gearbox_to_motor" type="fixed">
+      <origin xyz="-0.00555 0 0.19955" rpy="0 0 0"/>
+      <parent link="${tf_prefix}vention_rail_gearbox"/>
+      <child link="${tf_prefix}vention_rail_motor"/>
     </joint>
     <xacro:include filename="$(find vention_rail_description)/urdf/vention_rail.ros2_control.xacro" />

Commit message: added prismatic joint, need colors

File: vention_rail_description/urdf/vention_macro.urdf.xacro (robot description, xacro)
@@ -36,9 +36,9 @@
       </collision>
     </link>
-    <joint name="vention_rail_base_to_carriage" type="fixed">
+    <joint name="vention_rail_base_to_carriage" type="prismatic">
       <origin xyz="-0.96975 0 0.09600" rpy="0 0 0"/>
       <parent link="${tf_prefix}vention_rail_base_link"/>
       <child link="${tf_prefix}vention_rail_carriage"/>
-    </joint>
+      <limit lower="0" upper="${position_limit}" effort="1000" velocity="${velocity_limit}"/>
     <link name="${tf_prefix}vention_rail_gearbox">
       <visual>

Commit message: fixed bad tag

File: vention_rail_description/urdf/vention_macro.urdf.xacro (robot description, xacro)
@@ -41,4 +41,5 @@
       <child link="${tf_prefix}vention_rail_carriage"/>
       <limit lower="0" upper="${position_limit}" effort="1000" velocity="${velocity_limit}"/>
+    </joint>
     <link name="${tf_prefix}vention_rail_gearbox">
       <visual>

Commit message: added base joint internal to vention_macro.urdf.xacro, parent and origin parameters added and enabled

File: vention_rail_description/urdf/vention_macro.urdf.xacro (robot description, xacro)
@@ -4,4 +4,5 @@
     name
     tf_prefix
+    parent:=world
     use_fake_hardware:=false
     ip_addr:=192.168.1.104
@@ -9,5 +10,11 @@
     position_limit:=2.0
     velocity_limit:=0.15
-    acceleration_limit:=1.0">
+    acceleration_limit:=1.0
+    *origin">
+    <joint name="${tf_prefix}vention_rail_base_joint" type="fixed">
+      <parent link="${parent}"/>
+      <child link="${tf_prefix}vention_rail_base_link"/>
+      <xacro:insert_block name="origin"/>
+    </joint>
     <link name="${tf_prefix}vention_rail_base_link">
       <visual>

Commit message: moved to visual and changed from file to package

File: vention_rail_description/urdf/vention_macro.urdf.xacro (robot description, xacro)
@@ -21,5 +21,5 @@
         <origin xyz="0 0 0.045" rpy="0 0 0"/>
         <geometry>
-          <mesh filename="file://$(find vention_rail_description)/meshes/rail_des_live_body.dae"/>
+          <mesh filename="package://vention_rail_description/meshes/visual/rail_des_live_body.dae"/>
         </geometry>
       </visual>
@@ -34,5 +34,5 @@
       <visual>
         <geometry>
-          <mesh filename="file://$(find vention_rail_description)/meshes/rail_des_live_carriage.dae"/>
+          <mesh filename="package://vention_rail_description/meshes/visual/rail_des_live_carriage.dae"/>
         </geometry>
       </visual>
@@ -53,5 +53,5 @@
       <visual>
         <geometry>
-          <mesh filename="file://$(find vention_rail_description)/meshes/rail_des_gearbox.dae"/>
+          <mesh filename="package://vention_rail_description/meshes/visual/rail_des_gearbox.dae"/>
         </geometry>
       </visual>

Commit message: added visual and collision objects for vention rail motor cables

File: vention_rail_description/urdf/vention_macro.urdf.xacro (robot description, xacro)
@@ -85,4 +85,40 @@
       <child link="${tf_prefix}vention_rail_motor"/>
     </joint>
+    <link name="vention_rail_cable_0">
+      <visual>
+        <geometry>
+          <cylinder radius="0.015" length="0.075"/>
+        </geometry>
+      </visual>
+    </link>
+    <joint name="vention_motor_to_cable_0" type="fixed">
+      <origin xyz="0.0231 -0.0805 0.098" rpy="${radians(90)} 0 0"/>
+      <parent link="vention_rail_motor"/>
+      <child link="vention_rail_cable_0"/>
+    </joint>
+    <link name="vention_rail_cable_1">
+      <visual>
+        <geometry>
+          <cylinder radius="0.015" length="0.075"/>
+        </geometry>
+      </visual>
+    </link>
+    <joint name="vention_motor_to_cable_1" type="fixed">
+      <origin xyz="-0.0231 -0.0805 0.098" rpy="${radians(90)} 0 0"/>
+      <parent link="vention_rail_motor"/>
+      <child link="vention_rail_cable_1"/>
+    </joint>
+    <link name="vention_rail_cable_collision">
+      <collision>
+        <geometry>
+          <box size="0.0762 0.2286 0.0762"/>
+        </geometry>
+      </collision>
+    </link>
+    <joint name="vention_motor_to_cable_collision" type="fixed">
+      <origin xyz="0 -0.1573 0.0749" rpy="0 0 0"/>
+      <parent link="vention_rail_motor"/>
+      <child link="vention_rail_cable_collision"/>
+    </joint>
     <xacro:include filename="$(find vention_rail_description)/urdf/vention_rail.ros2_control.xacro" />
     <xacro:vention_rail_ros2_control

Commit message: added some missing tf_prefix calls to the rail macro

File: vention_rail_description/urdf/vention_macro.urdf.xacro (robot description, xacro)
@@ -44,5 +44,5 @@
       </collision>
     </link>
-    <joint name="vention_rail_base_to_carriage" type="prismatic">
+    <joint name="${tf_prefix}vention_rail_base_to_carriage" type="prismatic">
       <origin xyz="-0.96975 0 0.09600" rpy="0 0 0"/>
       <parent link="${tf_prefix}vention_rail_base_link"/>
@@ -63,10 +63,10 @@
       </collision>
     </link>
-    <joint name="vention_rail_base_to_gearbox" type="fixed">
+    <joint name="${tf_prefix}vention_rail_base_to_gearbox" type="fixed">
       <origin xyz="-1.3308 0 0.05455" rpy="0 0 0"/>
       <parent link="${tf_prefix}vention_rail_base_link"/>
       <child link="${tf_prefix}vention_rail_gearbox"/>
     </joint>
-    <link name="vention_rail_motor">
+    <link name="${tf_prefix}vention_rail_motor">
       <visual>
         <geometry>
@@ -80,10 +80,10 @@
       </collision>
     </link>
-    <joint name="vention_rail_gearbox_to_motor" type="fixed">
+    <joint name="${tf_prefix}vention_rail_gearbox_to_motor" type="fixed">
       <origin xyz="-0.00555 0 0.19955" rpy="0 0 0"/>
       <parent link="${tf_prefix}vention_rail_gearbox"/>
       <child link="${tf_prefix}vention_rail_motor"/>
     </joint>
-    <link name="vention_rail_cable_0">
+    <link name="${tf_prefix}vention_rail_cable_0">
       <visual>
         <geometry>
@@ -92,10 +92,10 @@
       </visual>
     </link>
-    <joint name="vention_motor_to_cable_0" type="fixed">
+    <joint name="${tf_prefix}vention_motor_to_cable_0" type="fixed">
       <origin xyz="0.0231 -0.0805 0.098" rpy="${radians(90)} 0 0"/>
-      <parent link="vention_rail_motor"/>
-      <child link="vention_rail_cable_0"/>
+      <parent link="${tf_prefix}vention_rail_motor"/>
+      <child link="${tf_prefix}vention_rail_cable_0"/>
     </joint>
-    <link name="vention_rail_cable_1">
+    <link name="${tf_prefix}vention_rail_cable_1">
       <visual>
         <geometry>
@@ -104,10 +104,10 @@
       </visual>
     </link>
-    <joint name="vention_motor_to_cable_1" type="fixed">
+    <joint name="${tf_prefix}vention_motor_to_cable_1" type="fixed">
       <origin xyz="-0.0231 -0.0805 0.098" rpy="${radians(90)} 0 0"/>
-      <parent link="vention_rail_motor"/>
-      <child link="vention_rail_cable_1"/>
+      <parent link="${tf_prefix}vention_rail_motor"/>
+      <child link="${tf_prefix}vention_rail_cable_1"/>
     </joint>
-    <link name="vention_rail_cable_collision">
+    <link name="${tf_prefix}vention_rail_cable_collision">
       <collision>
         <geometry>
@@ -116,8 +116,8 @@
       </collision>
     </link>
-    <joint name="vention_motor_to_cable_collision" type="fixed">
+    <joint name="${tf_prefix}vention_motor_to_cable_collision" type="fixed">
       <origin xyz="0 -0.1573 0.0749" rpy="0 0 0"/>
-      <parent link="vention_rail_motor"/>
-      <child link="vention_rail_cable_collision"/>
+      <parent link="${tf_prefix}vention_rail_motor"/>
+      <child link="${tf_prefix}vention_rail_cable_collision"/>
     </joint>
     <xacro:include filename="$(find vention_rail_description)/urdf/vention_rail.ros2_control.xacro" />

Commit message: Add inertia for base and carriage

File: vention_rail_description/urdf/vention_macro.urdf.xacro (robot description, xacro)
@@ -32,4 +32,8 @@
         </geometry>
       </collision>
+      <inertial>
+        <mass value="38.47"/>
+        <inertia ixx="0.46604111" ixy="0.0" ixz="0.0" iyy="0.46480515" iyz="-0.002668667" izz="0.1561"/>
+      </inertial>
     </link>
     <link name="${tf_prefix}vention_rail_carriage">
@@ -45,4 +49,8 @@
         </geometry>
       </collision>
+      <inertial>
+        <mass value="2.937"/>
+        <inertia ixx="0.0125" ixy="0.0" ixz="0.0" iyy="0.0287" iyz="0.0" izz="0.0199"/>
+      </inertial>
     </link>
     <joint name="${tf_prefix}vention_rail_base_to_carriage" type="prismatic">

Commit message: Add missing colors to a few objects in the description

File: vention_rail_description/urdf/vention_macro.urdf.xacro (robot description, xacro)
@@ -83,4 +83,7 @@
           <box size="0.086 0.086 0.226"/>
         </geometry>
+        <material name="${tf_prefix}vention_rail_motor">
+          <color rgba="0.8 0.8 0.8 1"/>
+        </material>
       </visual>
       <collision>
@@ -100,4 +103,7 @@
           <cylinder radius="0.015" length="0.075"/>
         </geometry>
+        <material name="${tf_prefix}vention_rail_cable_0">
+          <color rgba="0.8 0.8 0.8 1"/>
+        </material>
       </visual>
     </link>
@@ -112,4 +118,7 @@
           <cylinder radius="0.015" length="0.075"/>
         </geometry>
+        <material name="${tf_prefix}vention_rail_cable_1s">
+          <color rgba="0.8 0.8 0.8 1"/>
+        </material>
       </visual>
     </link>
